File: hardware/Reader/transceiver_sw_can.sch (KiCad schematic (older format))
At the start: 8 parts

Commit message: Revising reader
Parts:
- R_SWCAN_3: value 6.49k 0.12W -> 6.49k
Changed lines of the file:
@@
 Sheet 9 19
 Title "CANnect Reader | Single Wire CAN Transceiver"
-Date "2020-10-28"
-Rev "0.0.04"
+Date "2020-11-19"
+Rev "0.0.05"
 Comp "CANtech"
 Comment1 "Created by Choong Jin Ng | jin8383@gmail.com"
@@
 P 2850 2850
 F 0 "R_SWCAN_3" H 2909 2896 50  0000 L CNN
-F 1 "6.49k 0.12W" H 2909 2805 50  0000 L CNN
+F 1 "6.49k" H 2909 2805 50  0000 L CNN
 F 2 "footprints:RESC1608X55N" H 2850 2850 50  0001 C CNN
 F 3 "https://www.yageo.com/upload/media/product/productsearch/datasheet/rchip/PYu-RT_1-to-0.01_RoHS_L_12.pdf" H 2850 2850 50  0001 C CNN
